File: schematics/data_pod_battery_board/data_pod_battery_board.kicad_pcb (KiCad board)
At the start: 2 copper layers, 38 parts, among them J1 Conn_01x02, J10 Screw_Terminal_01x01, J11 Screw_Terminal_01x01, J12 Screw_Terminal_01x01, J13 Screw_Terminal_01x01, J14 Screw_Terminal_01x01, J15 Screw_Terminal_01x01, J16 Screw_Terminal_01x01, J17 Screw_Terminal_01x01, J18 Screw_Terminal_01x01, J19 Screw_Terminal_01x01, J2 Screw_Terminal_01x01, J20 Screw_Terminal_01x01, J21 Screw_Terminal_01x01, J22 Screw_Terminal_01x01, J23 Screw_Terminal_01x01, J24 Screw_Terminal_01x01, J25 Screw_Terminal_01x01, J26 Screw_Terminal_01x01, J27 Screw_Terminal_01x01, J28 Screw_Terminal_01x01, J29 Screw_Terminal_01x01, J3 Screw_Terminal_01x01, J30 Screw_Terminal_01x01, J31 Screw_Terminal_01x01, J32 Screw_Terminal_01x01, J33 Screw_Terminal_01x01, J34 Conn_01x02, J4 Screw_Terminal_01x01, J5 Screw_Terminal_01x01, J6 Screw_Terminal_01x01, J7 Screw_Terminal_01x01, J8 Screw_Terminal_01x01, J9 Screw_Terminal_01x01

Commit message: improved pcb outline
Parts:
- moved D1 584.2 mm to (617.2, 22.9)
- moved D2 584.2 mm to (684.8, 23.1)
- moved D3 584.2 mm to (752.9, 19.8)
- moved D4 584.2 mm to (842.3, 19.8)
- moved J1 584.2 mm to (981.2, 29.5)
- moved J10 584.2 mm to (615.2, 111.8)
- moved J11 584.2 mm to (684.3, 109.8)
- moved J12 584.2 mm to (762.0, 110.7)
- moved J13 584.2 mm to (842.6, 116.2)
- moved J15 584.2 mm to (681.0, 138.7)
- moved J17 584.2 mm to (840.0, 138.5)
- moved J18 584.2 mm to (614.4, 162.8)
- moved J19 584.2 mm to (680.7, 167.4)
- moved J2 584.2 mm to (614.4, 54.4)
- moved J21 584.2 mm to (841.0, 167.5)
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Routing:
- net (no net): vias 0 -> 48
Other:
- board outline added: 292.1 x 292.1 mm

Commit message: improved layout a little
Parts:
- added REF**: TL5937, battery:tl5937-tadiran 3.6v, B.Cu at (160.5, 282.1)
- added REF**: TL5937, battery:tl5937-tadiran 3.6v, B.Cu at (95.2, 135.1)
- added REF**: TL5937, battery:tl5937-tadiran 3.6v, B.Cu at (49.3, 135.1)
- added REF**: TL5937, battery:tl5937-tadiran 3.6v, B.Cu at (3.30, 135.1)
- added REF**: TL5937, battery:tl5937-tadiran 3.6v, F.Cu at (11.1, 185.7)
- added REF**: TL5937, battery:tl5937-tadiran 3.6v, F.Cu at (11.1, 231.7)
- added REF**: TL5937, battery:tl5937-tadiran 3.6v, F.Cu at (11.1, 277.7)
- added REF**: TL5937, battery:tl5937-tadiran 3.6v, F.Cu at (185.7, 282.0)
- added REF**: TL5937, battery:tl5937-tadiran 3.6v, F.Cu at (231.7, 282.0)
- added REF**: TL5937, battery:tl5937-tadiran 3.6v, F.Cu at (277.7, 282.0)
- added REF**: TL5937, battery:tl5937-tadiran 3.6v, F.Cu at (282.1, 108.0)
- added REF**: TL5937, battery:tl5937-tadiran 3.6v, B.Cu at (206.5, 282.1)
- added REF**: TL5937, battery:tl5937-tadiran 3.6v, F.Cu at (282.1, 62.0)
- added REF**: TL5937, battery:tl5937-tadiran 3.6v, F.Cu at (282.1, 16.0)
- added REF**: TL5937, battery:tl5937-tadiran 3.6v, F.Cu at (108.0, 10.0)
- added REF**: TL5937, battery:tl5937-tadiran 3.6v, F.Cu at (62.0, 10.0)
- added REF**: TL5937, battery:tl5937-tadiran 3.6v, F.Cu at (16.0, 10.0)
- added REF**: TL5937, battery:tl5937-tadiran 3.6v, B.Cu at (252.4, 282.1)
- added REF**: TL5937, battery:tl5937-tadiran 3.6v, B.Cu at (136.1, 198.5)
- added REF**: TL5937, battery:tl5937-tadiran 3.6v, B.Cu at (136.1, 244.5)
- added REF**: TL5937, battery:tl5937-tadiran 3.6v, B.Cu at (136.1, 290.4)
- added REF**: TL5937, battery:tl5937-tadiran 3.6v, B.Cu at (157.0, 95.2)
- added REF**: TL5937, battery:tl5937-tadiran 3.6v, B.Cu at (157.0, 49.2)
- added REF**: TL5937, battery:tl5937-tadiran 3.6v, B.Cu at (157.0, 3.25)
- J10, J14, J26, J30: moved to B.Cu
- moved D1 634.3 mm to (5.75, 191.7)
- moved J2 629.3 mm to (5.65, 213.9), turned to 90 degrees
- moved J18 616.2 mm to (5.79, 259.4), turned to 90 degrees
- moved J14 616.0 mm to (5.70, 226.1), turned to 90 degrees
- moved J30 608.8 mm to (5.95, 271.4), turned to 270 degrees
- moved J6 492.1 mm to (142.0, 214.1), turned to 90 degrees
- moved J10 487.0 mm to (141.7, 225.8), turned to 90 degrees
- moved J22 478.3 mm to (141.7, 256.8), turned to 90 degrees
- moved J26 475.0 mm to (141.6, 268.3), turned to 270 degrees
Routing:
- net (no net): vias 48 -> 49

Commit message: made some more changes to pcb
Parts:
- added D5: 1N5818, Diode_THT:D_DO-41_SOD81_P10.16mm_Horizontal, F.Cu at (201.9, 151.9)
- added D6: 1N5818, Diode_THT:D_DO-41_SOD81_P10.16mm_Horizontal, F.Cu at (288.3, 142.5)
- added J35: Screw_Terminal_01x01, terminals:screw_terminal_7.0mmx5.0mm, B.Cu at (179.6, 151.9)
- added J36: Screw_Terminal_01x01, terminals:screw_terminal_7.0mmx5.0mm, B.Cu at (271.0, 151.9)
- added J37: Screw_Terminal_01x01, terminals:screw_terminal_7.0mmx5.0mm, B.Cu at (179.8, 286.8)
- added J38: Screw_Terminal_01x01, terminals:screw_terminal_7.0mmx5.0mm, B.Cu at (271.8, 286.8)
- added J39: Screw_Terminal_01x01, terminals:screw_terminal_7.0mmx5.0mm, F.Cu at (166.9, 287.0)
- added J40: Screw_Terminal_01x01, terminals:screw_terminal_7.0mmx5.0mm, F.Cu at (258.6, 286.8)
- added J41: Screw_Terminal_01x01, terminals:screw_terminal_7.0mmx5.0mm, F.Cu at (166.1, 151.9)
- added J42: Screw_Terminal_01x01, terminals:screw_terminal_7.0mmx5.0mm, F.Cu at (257.8, 151.9)
- added J43: Screw_Terminal_01x01, terminals:screw_terminal_7.0mmx5.0mm, F.Cu at (287.5, 127.3)
- added J44: Screw_Terminal_01x01, terminals:screw_terminal_7.0mmx5.0mm, B.Cu at (225.8, 151.6)
- added J45: Screw_Terminal_01x01, terminals:screw_terminal_7.0mmx5.0mm, F.Cu at (151.6, 127.3)
- added J46: Screw_Terminal_01x01, terminals:screw_terminal_7.0mmx5.0mm, B.Cu at (225.3, 286.8)
- added J47: Screw_Terminal_01x01, terminals:screw_terminal_7.0mmx5.0mm, B.Cu at (151.4, 114.6)
- added J48: Screw_Terminal_01x01, terminals:screw_terminal_7.0mmx5.0mm, F.Cu at (212.6, 286.8)
- added J49: Screw_Terminal_01x01, terminals:screw_terminal_7.0mmx5.0mm, B.Cu at (287.0, 113.5)
- added J50: Screw_Terminal_01x01, terminals:screw_terminal_7.0mmx5.0mm, F.Cu at (212.6, 152.1)
- J11, J12, J13, J15, J16, J17, J27, J28, J29, J31, J32, J33: moved to B.Cu
- moved J32 749.8 mm to (67.6, 5.08)
- moved J29 718.7 mm to (151.6, 22.9), turned to 90 degrees
- moved J25 705.5 mm to (151.9, 36.3), turned to 90 degrees
- moved J28 701.3 mm to (68.3, 140.7)
- moved J20 700.7 mm to (80.6, 5.17)
- moved J13 692.1 mm to (152.1, 68.1), turned to 270 degrees
- moved J9 691.1 mm to (151.9, 81.5), turned to 90 degrees
- moved J31 690.7 mm to (5.08, 179.8), turned to 270 degrees
- moved J24 682.5 mm to (81.5, 141.0)
- moved J19 675.7 mm to (4.99, 166.7), turned to 270 degrees
- moved J15 672.7 mm to (21.7, 4.78)
- moved J11 662.7 mm to (22.4, 141.2)
- moved J16 660.0 mm to (113.0, 4.83)
- moved J3 652.5 mm to (35.1, 4.83)
- moved J7 650.3 mm to (35.6, 141.5)
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
Commit message: added more changes
Parts:
- J1, J34: footprint Connector_Molex:Molex_Mini-Fit_Sr_42819-22XX_1x02_P10.00mm_Vertical -> Connector_Molex:Molex_Nano-Fit_105309-xx02_1x02_P2.50mm_Vertical
- moved J1 126.0 mm to (393.2, 262.2), turned to 180 degrees
- moved J36 121.3 mm to (379.7, 205.7)
- moved J13 121.3 mm to (260.8, 121.9)
- moved J22 121.3 mm to (250.4, 312.1)
- moved J30 121.3 mm to (114.3, 326.3)
- moved J35 121.3 mm to (288.3, 205.7)
- moved J38 121.3 mm to (380.5, 340.6)
- moved J26 121.3 mm to (250.2, 325.6)
- moved J39 121.3 mm to (275.6, 340.8), turned to 180 degrees
- moved D2 121.3 mm to (167.1, 59.6)
- moved J10 121.3 mm to (250.4, 279.6)
- moved J19 121.3 mm to (113.7, 220.5), turned to 90 degrees
- moved J47 121.3 mm to (260.1, 168.4)
- moved REF** 121.3 mm to (307.1, 210.8)
- moved REF** 121.3 mm to (294.4, 335.8)
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
Commit message: finished battery baord pcb
Parts:
- moved J34 64.4 mm to (395.5, 262.2)
- moved J1 30.9 mm to (395.5, 293.1)
- moved D3 7.87 mm to (257.3, 58.3), turned to 180 degrees
- moved D2 1.66 mm to (166.2, 58.3)
- moved J25 1.43 mm to (260.1, 88.8)
- moved J6 1.35 mm to (250.4, 266.5)
- moved J16 1.29 mm to (223.0, 58.4)
- moved J2 1.23 mm to (114.4, 266.5)
- moved J7 1.14 mm to (143.7, 194.3)
- moved J30 1.11 mm to (114.4, 325.2)
- moved J42 1.00 mm to (367.4, 205.3)
- moved J49 0.89 mm to (396.2, 168.1)
- moved J32 0.89 mm to (177.0, 58.4)
- moved J37 0.83 mm to (288.1, 341.3)
- moved J13 0.81 mm to (260.1, 122.1)
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Connections:
- J10 pad : (no net) -> Net-(J10-Pad1)
- J11 pad : (no net) -> Net-(J11-Pad1)
- J12 pad : (no net) -> Net-(J12-Pad1)
- J13 pad : (no net) -> Net-(J13-Pad1)
- J14 pad : (no net) -> Net-(J14-Pad1)
- J15 pad : (no net) -> Net-(J15-Pad1)
- J16 pad : (no net) -> Net-(J16-Pad1)
- J17 pad : (no net) -> Net-(J17-Pad1)
- J18 pad : (no net) -> Net-(J14-Pad1)
- J19 pad : (no net) -> Net-(J15-Pad1)
- J2 pad : (no net) -> Net-(D1-Pad2)
- J20 pad : (no net) -> Net-(J16-Pad1)
- J21 pad : (no net) -> Net-(J17-Pad1)
- J22 pad : (no net) -> Net-(J22-Pad1)
- J23 pad : (no net) -> Net-(J23-Pad1)
- J24 pad : (no net) -> Net-(J24-Pad1)
- J25 pad : (no net) -> Net-(J25-Pad1)
- J26 pad : (no net) -> Net-(J22-Pad1)
- J27 pad : (no net) -> Net-(J23-Pad1)
- J28 pad : (no net) -> Net-(J24-Pad1)
- J29 pad : (no net) -> Net-(J25-Pad1)
- J3 pad : (no net) -> Net-(D2-Pad2)
- J30 pad : (no net) -> Net-(J30-Pad1)
- J31 pad : (no net) -> Net-(J30-Pad1)
- J32 pad : (no net) -> Net-(J30-Pad1)
- J33 pad : (no net) -> Net-(J30-Pad1)
- J35 pad : (no net) -> Net-(D5-Pad2)
- J36 pad : (no net) -> Net-(D6-Pad2)
- J37 pad : (no net) -> Net-(J37-Pad1)
- J38 pad : (no net) -> Net-(J38-Pad1)
- J39 pad : (no net) -> Net-(J37-Pad1)
- J4 pad : (no net) -> Net-(D3-Pad2)
- J40 pad : (no net) -> Net-(J38-Pad1)
- J41 pad : (no net) -> Net-(J41-Pad1)
- J42 pad : (no net) -> Net-(J42-Pad1)
- J43 pad : (no net) -> Net-(J41-Pad1)
- J44 pad : (no net) -> Net-(J42-Pad1)
- J45 pad : (no net) -> Net-(J45-Pad1)
- J46 pad : (no net) -> Net-(J46-Pad1)
- J47 pad : (no net) -> Net-(J45-Pad1)
- J48 pad : (no net) -> Net-(J46-Pad1)
- J49 pad : (no net) -> Net-(J30-Pad1)
- J5 pad : (no net) -> Net-(D4-Pad2)
- J50 pad : (no net) -> Net-(J30-Pad1)
- J6 pad : (no net) -> Net-(J10-Pad1)
- J7 pad : (no net) -> Net-(J11-Pad1)
- J8 pad : (no net) -> Net-(J12-Pad1)
- J9 pad : (no net) -> Net-(J13-Pad1)
Routing:
- net Net-(J30-Pad1): track 0.00 -> 1172.3 mm
- net Net-(D1-Pad1): track 0.00 -> 807.3 mm
- net Net-(J15-Pad1): track 0.00 -> 209.0 mm
- net Net-(J41-Pad1): track 0.00 -> 186.7 mm
- net Net-(J1-Pad2): track 0.00 -> 105.4 mm
- net Net-(J14-Pad1): track 0.00 -> 100.8 mm
- net Net-(J42-Pad1): track 0.00 -> 95.8 mm
- net Net-(J46-Pad1): track 0.00 -> 78.0 mm
- net Net-(J17-Pad1): track 0.00 -> 77.2 mm
- net Net-(J38-Pad1): track 0.00 -> 76.3 mm
- net Net-(J37-Pad1): track 0.00 -> 66.4 mm
- net Net-(J16-Pad1): track 0.00 -> 61.5 mm
- net Net-(J45-Pad1): track 0.00 -> 59.8 mm
- net Net-(J13-Pad1): track 0.00 -> 59.6 mm
- net Net-(J10-Pad1): track 0.00 -> 59.5 mm
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