File: schematics/datapod/_autosave-datapod_5v_power.sch (KiCad schematic (older format))
At the start: 11 parts, among them J7 Conn_02x02_Odd_Even, U5 LT1374CS8-5PBF

Commit message: added rtc stuff , rotated db9s , added on/off transistors for max chip and sdcard
Parts:
- D5: Part# 1514-CMDSH-3TRPBFREETR-ND -> 1514-CMDSH-3TRPBFREECT-ND
Changed lines of the file:
@@
 F 3 "https://my.centralsemi.com/get_document.php?cmp=1&mergetype=pd&mergepath=pd&pdf_id=CMDSH-3.PDF" H 9900 2600 50  0001 C CNN
 F 4 "Digikey" H 9900 2600 50  0001 C CNN "Vendor"
-F 5 "1514-CMDSH-3TRPBFREETR-ND" H 9900 2600 50  0001 C CNN "Part#"
+F 5 "1514-CMDSH-3TRPBFREECT-ND" H 9900 2600 50  0001 C CNN "Part#"
 	1    9900 2600
 	1    0    0    -1
