File: schematics/datapod/datapod_5v_power.sch (KiCad schematic (older format))
At the start: 11 parts, among them J7 Conn_02x02_Odd_Even, U5 LT1374CS8-5PBF

Commit message: rev 3 , moved db9 connectors out and added ajumper to change output to 14.4v
Parts:
- TP1: Part# (none) -> DNI
- U5: Field4 SO-8 Linear Technology -> (none); Field5 https://www.digikey.com/product-detail/en/linear-technology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 -> (none); Field6 LT1374 - 4.5A, 500kHz Step-Down Switching Regulator -> (none); Field7 LT1374CS8-5#PBF -> (none); Vendor (none) -> Digikey
Changed lines of the file:
@@
 F 2 "Package_SO:SO-8_3.9x4.9mm_P1.27mm" H 4725 4450 50  0001 L BNN
 F 3 "Linear Technology" H 4700 3875 50  0001 L BNN
-F 4 "SO-8 Linear Technology" H 4650 4050 50  0001 L BNN "Field4"
-F 5 "https://www.digikey.com/product-detail/en/linear-technology-analog-devices/LT1374CS8-5-PBF/LT1374CS8-5-PBF-ND/888771?utm_source=snapeda&utm_medium=aggregator&utm_campaign=symbol" H 4675 3600 50  0001 L BNN "Field5"
-F 6 "LT1374 - 4.5A, 500kHz Step-Down Switching Regulator" H 4675 3725 50  0001 L BNN "Field6"
-F 7 "LT1374CS8-5#PBF" H 4700 4175 50  0001 L BNN "Field7"
-F 8 "LT1374CS8-5#PBF-ND" H 4725 4300 50  0001 L BNN "Part#"
+F 4 "LT1374CS8-5#PBF-ND" H 4725 4300 50  0001 L BNN "Part#"
+F 5 "Digikey" H 4400 3050 50  0001 C CNN "Vendor"
 	1    4400 3050
 	1    0    0    -1
@@
 F 2 "TestPoint:TestPoint_2Pads_Pitch5.08mm_Drill1.3mm" H 9300 950 50  0001 C CNN
 F 3 "~" H 9300 950 50  0001 C CNN
+F 4 "DNI" H 9300 950 50  0001 C CNN "Part#"
 	1    9300 950
 	-1   0    0    1
