File: schematics/datapod/datapods_sdcard.sch (KiCad schematic (older format))
At the start: 3 parts, among them J6 Micro_SD_Card, U3 74LVC125

Commit message: added rtc stuff , rotated db9s , added on/off transistors for max chip and sdcard
Parts:
- added Q5: FDG1024NZ, Package_TO_SOT_SMD:SOT-363_SC-70-6, symbol Transistor_FET:FDG1024NZ
Connections:
- net GND: now also Q5.1 (S), Q5.4 (S); no longer J6.6 (VSS), U3.7 (GND)
- new net: Q5.6 (D), U3.7 (GND)
- new net: J6.6 (VSS), Q5.3 (D)
- new net uSD_ON_OFF: Q5.2 (G), Q5.5 (G)
Changed lines of the file:
@@
 L power:GND #PWR031
 U 1 1 5E4DF563
-P 1500 3450
-F 0 "#PWR031" H 1500 3200 50  0001 C CNN
-F 1 "GND" H 1505 3277 50  0000 C CNN
-F 2 "" H 1500 3450 50  0001 C CNN
-F 3 "" H 1500 3450 50  0001 C CNN
-	1    1500 3450
+P 1500 6450
+F 0 "#PWR031" H 1500 6200 50  0001 C CNN
+F 1 "GND" H 1505 6277 50  0000 C CNN
+F 2 "" H 1500 6450 50  0001 C CNN
+F 3 "" H 1500 6450 50  0001 C CNN
+	1    1500 6450
 	1    0    0    -1
 $EndComp
 Wire Wire Line
 	1500 2000 1500 2200
-Wire Wire Line
-	1500 3200 1500 3450
 NoConn ~ 7750 3100
 NoConn ~ 7750 3800
@@
 L power:GND #PWR033
 U 1 1 5E4E4242
-P 7500 4450
-F 0 "#PWR033" H 7500 4200 50  0001 C CNN
-F 1 "GND" H 7505 4277 50  0000 C CNN
-F 2 "" H 7500 4450 50  0001 C CNN
-F 3 "" H 7500 4450 50  0001 C CNN
-	1    7500 4450
+P 9450 4650
+F 0 "#PWR033" H 9450 4400 50  0001 C CNN
+F 1 "GND" H 9455 4477 50  0000 C CNN
+F 2 "" H 9450 4650 50  0001 C CNN
+F 3 "" H 9450 4650 50  0001 C CNN
+	1    9450 4650
 	1    0    0    -1
 $EndComp
 Wire Wire Line
 	7750 3600 7500 3600
-Wire Wire Line
-	7500 3600 7500 4300
 Wire Wire Line
 	7750 3400 7500 3400
@@
 Wire Wire Line
 	4950 2250 5600 2250
-Wire Wire Line
-	9450 4300 7500 4300
-Connection ~ 7500 4300
-Wire Wire Line
-	7500 4300 7500 4450
 $Comp
 L 74xx:74LVC125 U3
@@
 	1    0    0    -1
 $EndComp
-Wire Wire Line
-	9450 4000 9450 4300
 Text Notes 9650 3600 0    59   ~ 0
 DAT2/X\nDAT3/CS\nCMD/DI\nVDD/VDD\nCLK/SCLK\nVSS/VSS\nDAT0/ D0\nDAT1/ X
@@
 	4950 1950 4950 2250
 Connection ~ 4950 2250
-Wire Wire Line
-	4950 1450 4950 1500
 $Comp
 L power:+5V #PWR?
@@
 	1    0    0    -1
 $EndComp
-Connection ~ 4950 1500
-Wire Wire Line
-	4950 1500 4950 1650
+Wire Wire Line
+	4950 1450 4950 1650
+$Comp
+L Transistor_FET:FDG1024NZ Q5
+U 1 1 5E240480
+P 1600 6050
+F 0 "Q5" H 1450 6300 50  0000 L CNN
+F 1 "FDG1024NZ" H 1900 5950 50  0000 L CNN
+F 2 "Package_TO_SOT_SMD:SOT-363_SC-70-6" H 1800 5975 50  0001 L CIN
+F 3 "http://www.fairchildsemi.com/ds/FD/FDG1024NZ.pdf" H 1600 6050 50  0001 L CNN
+F 4 "Digikey" H 1600 6050 50  0001 C CNN "Vendor"
+F 5 "FDG1024NZFSCT-ND" H 1600 6050 50  0001 C CNN "Part#"
+	1    1600 6050
+	-1   0    0    -1
+$EndComp
+$Comp
+L Transistor_FET:FDG1024NZ Q5
+U 2 1 5E245C91
+P 7600 5400
+F 0 "Q5" H 7450 5600 50  0000 L CNN
+F 1 "FDG1024NZ" H 7150 5200 50  0000 L CNN
+F 2 "Package_TO_SOT_SMD:SOT-363_SC-70-6" H 7800 5325 50  0001 L CIN
+F 3 "http://www.fairchildsemi.com/ds/FD/FDG1024NZ.pdf" H 7600 5400 50  0001 L CNN
+F 4 "Digikey" H 7600 5400 50  0001 C CNN "Vendor"
+F 5 "FDG1024NZFSCT-ND" H 7600 5400 50  0001 C CNN "Part#"
+	2    7600 5400
+	-1   0    0    -1
+$EndComp
+Wire Wire Line
+	1500 6250 1500 6450
+Wire Wire Line
+	1500 3200 1500 5850
+$Comp
+L power:GND #PWR0114
+U 1 1 5E28125B
+P 7500 5900
+F 0 "#PWR0114" H 7500 5650 50  0001 C CNN
+F 1 "GND" H 7505 5727 50  0000 C CNN
+F 2 "" H 7500 5900 50  0001 C CNN
+F 3 "" H 7500 5900 50  0001 C CNN
+	1    7500 5900
+	1    0    0    -1
+$EndComp
+Wire Wire Line
+	9450 4000 9450 4650
+Wire Wire Line
+	7500 3600 7500 4950
+Wire Wire Line
+	7500 5600 7500 5900
+Text GLabel 2100 6050 2    50   Input ~ 0
+uSD_ON_OFF
+Text GLabel 8200 5400 2    50   Input ~ 0
+uSD_ON_OFF
+Wire Wire Line
+	1800 6050 2100 6050
+Wire Wire Line
+	7800 5400 8200 5400
+$Comp
+L power:PWR_FLAG #FLG0107
+U 1 1 5E2CC5A0
+P 900 5450
+F 0 "#FLG0107" H 900 5525 50  0001 C CNN
+F 1 "PWR_FLAG" H 900 5623 50  0000 C CNN
+F 2 "" H 900 5450 50  0001 C CNN
+F 3 "~" H 900 5450 50  0001 C CNN
+	1    900  5450
+	1    0    0    -1
+$EndComp
+Wire Wire Line
+	900  5450 900  5850
+Wire Wire Line
+	900  5850 1500 5850
+Connection ~ 1500 5850
+$Comp
+L power:PWR_FLAG #FLG0108
+U 1 1 5E2CE293
+P 8250 4750
+F 0 "#FLG0108" H 8250 4825 50  0001 C CNN
+F 1 "PWR_FLAG" H 8250 4923 50  0000 C CNN
+F 2 "" H 8250 4750 50  0001 C CNN
+F 3 "~" H 8250 4750 50  0001 C CNN
+	1    8250 4750
+	1    0    0    -1
+$EndComp
+Wire Wire Line
+	8250 4750 8250 4950
+Wire Wire Line
+	8250 4950 7500 4950
+Connection ~ 7500 4950
+Wire Wire Line
+	7500 4950 7500 5200
 $EndSCHEMATC

Commit message: added a fabrication file, updated gerbers to include fab masks, and updated R5 part number
Parts:
- R5: part# 749-1125-6-ND -> 311-10KERCT-ND
Changed lines of the file:
@@
 F 1 "10K" H 5020 1755 50  0000 L CNN
 F 2 "Resistor_SMD:R_1206_3216Metric_Pad1.42x1.75mm_HandSolder" V 4880 1800 50  0001 C CNN
-F 3 "http://www.vishay.com/docs/28796/mcw0406atpro.pdf" H 4950 1800 50  0001 C CNN
+F 3 "https://www.yageo.com/upload/media/product/productsearch/datasheet/rchip/PYu-RC_Group_51_RoHS_L_10.pdf" H 4950 1800 50  0001 C CNN
 F 4 "Digikey" H 4950 1800 50  0001 C CNN "Vendor"
-F 5 "749-1125-6-ND" H 4950 1800 50  0001 C CNN "part#"
+F 5 "311-10KERCT-ND" H 4950 1800 50  0001 C CNN "part#"
 	1    4950 1800
 	1    0    0    -1

Commit message: rev 3 , moved db9 connectors out and added ajumper to change output to 14.4v
Parts:
- R5: Part# (none) -> 311-10KERCT-ND; part# 311-10KERCT-ND -> (none)
Changed lines of the file:
@@
 F 3 "https://www.yageo.com/upload/media/product/productsearch/datasheet/rchip/PYu-RC_Group_51_RoHS_L_10.pdf" H 4950 1800 50  0001 C CNN
 F 4 "Digikey" H 4950 1800 50  0001 C CNN "Vendor"
-F 5 "311-10KERCT-ND" H 4950 1800 50  0001 C CNN "part#"
+F 5 "311-10KERCT-ND" H 4950 1800 50  0001 C CNN "Part#"
 	1    4950 1800
 	1    0    0    -1
