File: schematics/datapod/datapod_serial.sch (KiCad schematic (older format))
At the start: 11 parts, among them J4 DB9_Female, J5 DB9_Male_MountingHoles, Q3 IRF7324, Q4 FDG1024NZ, U2 MAX232

Commit message: added two capacitors
Parts:
- JP2: Part# (none) -> DNI
Changed lines of the file:
@@
 F 2 "Jumper:SolderJumper-3_P1.3mm_Open_RoundedPad1.0x1.5mm" H 5750 5700 50  0001 C CNN
 F 3 "~" H 5750 5700 50  0001 C CNN
+F 4 "DNI" V 5750 5700 50  0001 C CNN "Part#"
 	1    5750 5700
 	0    1    1    0
